Commit message: ros2 control

File: urdf/bolt.xacro (robot description, xacro)
@@ -6,4 +6,10 @@
   xmlns:xacro="http://playerstage.sourceforge.net/gazebo/xmlschema/#interface">
   <xacro:macro name="bolt_full" params="mesh_ext color_name color opacity new_leg has_passive_ankle">
+    <gazebo>
+      <plugin filename="libgz_ros2_control-system.so" name="gz_ros2_control::GazeboSimROS2ControlPlugin">
+        <parameters>$(find bolt_visu)/config/bolt_gz_controller.yaml</parameters>
+        <controller_manager_prefix_node_name>controller_manager</controller_manager_prefix_node_name>
+      </plugin>
+    </gazebo>
     <!-- This file is based on: https://atlas.is.localnet/confluence/display/AMDW/Quadruped+URDF+Files -->
     <link name="base_link">

File: urdf/leg.xacro (robot description, xacro)
@@ -24,4 +24,20 @@
                                     mesh_ext color_name color opacity new_leg
                                     has_passive_ankle">
+        <ros2_control name="GazeboSimSystem" type="system">
+          <hardware>
+            <plugin>gz_ros2_control/GazeboSimSystem</plugin>
+          </hardware>
+          <joint name="${prefix}_HAA">
+            <command_interface name="effort">
+              <param name="min">-1000</param>
+              <param name="max">1000</param>
+            </command_interface>
+            <state_interface name="position">
+              <param name="initial_value">1.0</param>
+            </state_interface>
+            <state_interface name="velocity"/>
+            <state_interface name="effort"/>
+          </joint>
+        </ros2_control>
         <joint name="${prefix}_HAA" type="revolute">
             <parent link="base_link"/>
@@ -37,10 +53,4 @@
                 <origin xyz="${base_2_HAA_x} ${-base_2_HAA_y} 0" rpy="0 0 0"/>
             </xacro:if>
-            <!--xacro:unless value="${is_right}">
-        <origin xyz="${base_2_HAA_x} ${base_2_HAA_y + 0.0007888} ${-base_2_HAA_z}" rpy="0 0 0" />
-      </xacro:unless>
-      <xacro:if value="${is_right}">
-        <origin xyz="${base_2_HAA_x} ${-base_2_HAA_y + 0.0007888} ${-base_2_HAA_z}" rpy="0 0 0" />
-      </xacro:if-->
             <!-- pybullet simulation parameters -->
             <dynamics damping="0.0" friction="0.0"/>
