Commit message: position controller

File: urdf/bolt.urdf.xacro (robot description, xacro)
@@ -13,4 +13,6 @@
   <!-- Include the legs -->
   <xacro:include filename="bolt.xacro"/>
+  <!-- Include the joint_interface -->
+  <xacro:include filename="joint_interface.xacro"/>
   <!-- Include the fully parametrized bolt -->
   <xacro:bolt_full
@@ -21,3 +23,19 @@
       new_leg="${new_leg}"
       has_passive_ankle="${has_passive_ankle}"/>
+  <gazebo>
+    <plugin filename="libgz_ros2_control-system.so" name="gz_ros2_control::GazeboSimROS2ControlPlugin">
+      <parameters>$(find bolt_visu)/config/bolt_gz_controller.yaml</parameters>
+    </plugin>
+  </gazebo>
+  <ros2_control name="GazeboSymSystem" type="system">
+    <hardware>
+      <plugin>gz_ros2_control/GazeboSimSystem</plugin>
+    </hardware>
+    <xacro:joint_interface name="FR_HAA" p="10" d="0.1" t="1"/>
+    <xacro:joint_interface name="FR_HFE" p="10" d="0.1" t="1"/>
+    <xacro:joint_interface name="FR_KFE" p="10" d="0.1" t="1"/>
+    <xacro:joint_interface name="FL_HAA" p="10" d="0.1" t="1"/>
+    <xacro:joint_interface name="FL_HFE" p="10" d="0.1" t="1"/>
+    <xacro:joint_interface name="FL_KFE" p="10" d="0.1" t="1"/>
+  </ros2_control>
 </robot>

File: urdf/bolt.xacro (robot description, xacro)
@@ -6,10 +6,4 @@
   xmlns:xacro="http://playerstage.sourceforge.net/gazebo/xmlschema/#interface">
   <xacro:macro name="bolt_full" params="mesh_ext color_name color opacity new_leg has_passive_ankle">
-    <gazebo>
-      <plugin filename="libgz_ros2_control-system.so" name="gz_ros2_control::GazeboSimROS2ControlPlugin">
-        <parameters>$(find bolt_visu)/config/bolt_gz_controller.yaml</parameters>
-        <controller_manager_prefix_node_name>controller_manager</controller_manager_prefix_node_name>
-      </plugin>
-    </gazebo>
     <!-- This file is based on: https://atlas.is.localnet/confluence/display/AMDW/Quadruped+URDF+Files -->
     <link name="base_link">

File: urdf/leg.xacro (robot description, xacro)
@@ -24,20 +24,4 @@
                                     mesh_ext color_name color opacity new_leg
                                     has_passive_ankle">
-        <ros2_control name="GazeboSimSystem" type="system">
-          <hardware>
-            <plugin>gz_ros2_control/GazeboSimSystem</plugin>
-          </hardware>
-          <joint name="${prefix}_HAA">
-            <command_interface name="effort">
-              <param name="min">-1000</param>
-              <param name="max">1000</param>
-            </command_interface>
-            <state_interface name="position">
-              <param name="initial_value">1.0</param>
-            </state_interface>
-            <state_interface name="velocity"/>
-            <state_interface name="effort"/>
-          </joint>
-        </ros2_control>
         <joint name="${prefix}_HAA" type="revolute">
             <parent link="base_link"/>
